Commit message: 플로팅 로봇 팩 1.0.4: 얼굴 질량 180 → 245 kg (구 65 kg 포함 · 구 메쉬 없이 얼굴 쉘에 합산)
- model.xml · robot.urdf: pitch 바디 260.8 → 325.8 kg (무게중심·관성 재계산)
- 4대 모두 sim_run --check 통과

Co-Authored-By: Claude Opus 5.5 <noreply@anthropic.com>

File: floating_narration_all/robot_pack_1/robot.urdf (robot description, URDF)
Before this commit: robot floating_head_1800, 6 links, 5 joints
Links:
- link pitch: mass 260.8240 -> 325.8240

Commit message: 플로팅 로봇 팩 1.0.5: 눈 링크 구조 반영 (유니버설 조인트 + 4절 링크)
- Fusion 확인: 눈알은 구 중심의 UNKA12 유니버설 조인트 위 · 상하 = KHY55 크랭크 54 mm → 로드 132 mm,
  좌우 = PGX44 암 90 mm → 로드 72 mm
- 모터 관절 이름 그대로 (값 = 감속기 출력각 = Blender 본 값) · eye_pitch 축을 KHY55 출력축으로
- 눈알 관절 eyeball_pitch_* / eyeball_yaw_* 추가 · equality polycoef (4절 링크 3차 근사, 오차 0.003°)
  눈 상하 ≈ 0.56배 · 좌우 ≈ 0.955배
- 링크로 이어진 눈알 관성을 모터 관절 armature 에 더함 (실행기 게인 = 관절 자기 관성 기준)
- 나레이션 시뮬: 눈 상하 정지 41.6 → 13.2 Nm · 최대 17.7 Nm (T2N 51%) · 오차 0.03°
- 4대 모두 sim_run --check 통과

Co-Authored-By: Claude Opus 5.5 <noreply@anthropic.com>

File: floating_narration_all/robot_pack_1/robot.urdf (robot description, URDF)
Before this commit: robot floating_head_1800, 6 links, 5 joints
Links:
- added link eyeball_l, mass 20.1981; visual mesh filename=meshes/eyeball_l_0.stl
- added link eyeball_pitch_l, mass 0.0100
- added link eyeball_pitch_r, mass 0.0100
- added link eyeball_r, mass 20.1981; visual mesh filename=meshes/eyeball_r_0.stl
- link eye_yaw_l: mass 20.3657 -> 0.0836
- link eye_yaw_r: mass 20.4744 -> 0.0836
- link pitch: mass 325.8240 -> 325.9920
Joints:
- added joint eyeball_pitch_l: type revolute, parent pitch, child eyeball_pitch_l, origin xyz=0.268 -0.3683 -0.0444 rpy=0 0 0, axis -0.995194 -0.0810158 -0.0550107, limit lower=-0.5 upper=0.5 effort=0 velocity=10, mimic joint=eye_pitch multiplier=0.5600 offset=0
- added joint eyeball_pitch_r: type revolute, parent pitch, child eyeball_pitch_r, origin xyz=-0.268 -0.3683 -0.0444 rpy=0 0 0, axis -0.995194 0.0810158 0.0550107, limit lower=-0.5 upper=0.5 effort=0 velocity=10, mimic joint=eye_pitch multiplier=0.5600 offset=0
- added joint eyeball_yaw_l: type revolute, parent eyeball_pitch_l, child eyeball_l, origin xyz=0 0 0 rpy=0 0 0, axis 0 -0.559215 0.829023, limit lower=-0.5 upper=0.5 effort=0 velocity=10, mimic joint=eye_yaw_l multiplier=0.9554 offset=0
- added joint eyeball_yaw_r: type revolute, parent eyeball_pitch_r, child eyeball_r, origin xyz=0 0 0 rpy=0 0 0, axis 0 -0.559215 0.829023, limit lower=-0.5 upper=0.5 effort=0 velocity=10, mimic joint=eye_yaw_r multiplier=0.9554 offset=0
- joint eye_pitch: axis -1 0 0 -> 1 0 0; origin xyz=0 -0.3231 -0.0117 rpy=0 0 0 -> xyz=0 -0.355 0.115 rpy=0 0 0
- joint eye_yaw_l: origin xyz=0.2625 0 0 rpy=0 0 0 -> xyz=0.2625 -0.3241 -0.0103 rpy=0 0 0; parent eye_pitch -> pitch
- joint eye_yaw_r: origin xyz=-0.2625 0 0 rpy=0 0 0 -> xyz=-0.2625 -0.3241 -0.0103 rpy=0 0 0; parent eye_pitch -> pitch
