Commit message: packs 1.0.10: per-robot designer face/eye meshes (gray); narration neck pitch scaled x0.8 (max 10 deg)
- floating_narration_all_9min/_90s: neck pitch keys x0.8 in the .blend (no clamping), re-exported; max 10.0 deg, export check errors 0
- floatingN_pack: meshes/face.stl, eyeball_l/r.stl from the designer head at that spot (Blender decimate, 30k/5k tris), replaces pitch_0/eyeball_*_0; inertials unchanged
- scene.glb rebuilt from the scaled animation

Co-Authored-By: Claude Opus 5.5 <noreply@anthropic.com>

File: floating1_pack/robot.urdf (robot description, URDF)
Before this commit: robot floating_head_1800, 10 links, 9 joints
Links:
- link eyeball_l: geometry visual mesh filename=meshes/eyeball_l.stl
- link eyeball_r: geometry visual mesh filename=meshes/eyeball_r.stl
- link pitch: geometry visual mesh filename=meshes/face.stl

Commit message: packs 1.0.11: 로봇별 얼굴 무게중심·관성 · 눈알 회전 중심
- 얼굴 245 kg 그대로 · 무게중심·관성을 그 로봇 디자이너 얼굴(face.stl) 균일 껍질로 (1.0.10 까지 1800 Fusion 얼굴)
- 눈알 U-조인트 중심 = Blender 리그 눈 본 머리 (x ±243.9 / 236.8 / 248.2 / 277.1 mm · y −381 · z 157.2) · 눈알 바디 같이 이동
- 링크 비율 · 질량 · 기구는 그대로 · model.xml · robot.urdf · sim_run --check 4개 OK

Co-Authored-By: Claude Opus 5.5 <noreply@anthropic.com>

File: floating1_pack/robot.urdf (robot description, URDF)
Before this commit: robot floating_head_1800, 10 links, 9 joints
Joints:
- joint eyeball_pitch_l: origin xyz=0.268 -0.3683 -0.0444 rpy=0 0 0 -> xyz=0.2439 -0.381 -0.0116 rpy=0 0 0
- joint eyeball_pitch_r: origin xyz=-0.268 -0.3683 -0.0444 rpy=0 0 0 -> xyz=-0.2439 -0.381 -0.0116 rpy=0 0 0

File: floating2_pack/robot.urdf (robot description, URDF)
Before this commit: robot floating_head_1800, 10 links, 9 joints
Joints:
- joint eyeball_pitch_l: origin xyz=0.268 -0.3683 -0.0444 rpy=0 0 0 -> xyz=0.2368 -0.381 -0.0116 rpy=0 0 0
- joint eyeball_pitch_r: origin xyz=-0.268 -0.3683 -0.0444 rpy=0 0 0 -> xyz=-0.2368 -0.381 -0.0116 rpy=0 0 0

File: floating3_pack/robot.urdf (robot description, URDF)
Before this commit: robot floating_head_1800, 10 links, 9 joints
Joints:
- joint eyeball_pitch_l: origin xyz=0.268 -0.3683 -0.0444 rpy=0 0 0 -> xyz=0.2482 -0.381 -0.0116 rpy=0 0 0
- joint eyeball_pitch_r: origin xyz=-0.268 -0.3683 -0.0444 rpy=0 0 0 -> xyz=-0.2482 -0.381 -0.0116 rpy=0 0 0

File: floating4_pack/robot.urdf (robot description, URDF)
Before this commit: robot floating_head_1800, 10 links, 9 joints
Joints:
- joint eyeball_pitch_l: origin xyz=0.268 -0.3683 -0.0444 rpy=0 0 0 -> xyz=0.2771 -0.381 -0.0116 rpy=0 0 0
- joint eyeball_pitch_r: origin xyz=-0.268 -0.3683 -0.0444 rpy=0 0 0 -> xyz=-0.2771 -0.381 -0.0116 rpy=0 0 0
