Commit message: la 팩 1.0.0 (f2 · f3 · f4) · ny 팩 1.0.15 (배치 f2 · f4 · f3) (2026-10-19)
옛 기록: fdda910..a9a9fd3 (커밋 2개) · y0ung-GMLAB/animation_robot_pack-archive

File: ny/floating1_pack/robot.urdf (robot description, URDF)
Before this commit: robot floating_head_1800, 10 links, 9 joints
Joints:
- joint eyeball_pitch_l: origin xyz=0.2439 -0.381 -0.0116 rpy=0 0 0 -> xyz=0.2771 -0.381 -0.0116 rpy=0 0 0
- joint eyeball_pitch_r: origin xyz=-0.2439 -0.381 -0.0116 rpy=0 0 0 -> xyz=-0.2771 -0.381 -0.0116 rpy=0 0 0

File: ny/floating2_pack/robot.urdf (robot description, URDF)
Before this commit: robot floating_head_1800, 10 links, 9 joints
Joints:
- joint eyeball_pitch_l: origin xyz=0.2368 -0.381 -0.0116 rpy=0 0 0 -> xyz=0.2439 -0.381 -0.0116 rpy=0 0 0
- joint eyeball_pitch_r: origin xyz=-0.2368 -0.381 -0.0116 rpy=0 0 0 -> xyz=-0.2439 -0.381 -0.0116 rpy=0 0 0

File: ny/floating4_pack/robot.urdf (robot description, URDF)
Before this commit: robot floating_head_1800, 10 links, 9 joints
Joints:
- joint eyeball_pitch_l: origin xyz=0.2771 -0.381 -0.0116 rpy=0 0 0 -> xyz=0.2368 -0.381 -0.0116 rpy=0 0 0
- joint eyeball_pitch_r: origin xyz=-0.2771 -0.381 -0.0116 rpy=0 0 0 -> xyz=-0.2368 -0.381 -0.0116 rpy=0 0 0
