Commit message: 고개 좌우 가동범위 ±15 → ±18 · ny 팩 1.0.16 · la 팩 1.0.1 (2026-10-27)
옛 기록: 368f6db..368f6db (커밋 1개) · y0ung-GMLAB/animation_robot_pack-archive

File: floating/floating1_pack/robot.urdf (robot description, URDF)
Before this commit: robot floating_head_1800, 10 links, 9 joints
Joints:
- joint neck_yaw: limit lower=-0.26180 upper=0.26180 effort=644.4 velocity=0.3840 -> lower=-0.31416 upper=0.31416 effort=644.4 velocity=0.3840

File: floating/floating2_pack/robot.urdf (robot description, URDF)
Before this commit: robot floating_head_1800, 10 links, 9 joints
Joints:
- joint neck_yaw: limit lower=-0.26180 upper=0.26180 effort=644.4 velocity=0.3840 -> lower=-0.31416 upper=0.31416 effort=644.4 velocity=0.3840

File: floating/floating3_pack/robot.urdf (robot description, URDF)
Before this commit: robot floating_head_1800, 10 links, 9 joints
Joints:
- joint neck_yaw: limit lower=-0.26180 upper=0.26180 effort=644.4 velocity=0.3840 -> lower=-0.31416 upper=0.31416 effort=644.4 velocity=0.3840

File: floating/floating4_pack/robot.urdf (robot description, URDF)
Before this commit: robot floating_head_1800, 10 links, 9 joints
Joints:
- joint neck_yaw: limit lower=-0.26180 upper=0.26180 effort=644.4 velocity=0.3840 -> lower=-0.31416 upper=0.31416 effort=644.4 velocity=0.3840
